Commit message: data

File: multirobot_simulation/ares_description/urdf/ares_laser.xacro (robot description, xacro)
@@ -24,5 +24,5 @@
         <origin xyz="${camera_offset_x} ${camera_offset_y} ${camera_offset_z}" rpy="0 0 0" />
         <parent link="base_link"/>
-        <child link="imu_sensor_link"/>
+        <child link="imu_sensor_link"/>`
     </joint>
     <xacro:imu_sensor prefix="imu_sensor"/>

File: multirobot_simulation/ares_description/urdf/sensors/camera.xacro (robot description, xacro)
@@ -34,7 +34,7 @@
                     <horizontal_fov>1.3962634</horizontal_fov>
                     <image>
-                        <width>1280</width>
-                        <height>720</height>
-                        <format>R8G8B8</format>
+                        <width>752</width>
+                        <height>480</height>
+                        <format>L8</format>
                     </image>
                     <clip>

File: multirobot_simulation/ares_description/urdf/sensors/imu_o.xacro (robot description, xacro)
@@ -39,5 +39,5 @@
 		<bodyName>imu_sensor_link</bodyName>
 		<updateRateHZ>100.0</updateRateHZ>
-		<gaussianNoise>1.0</gaussianNoise>
+		<gaussianNoise>0.0</gaussianNoise>
 		<xyzOffset>0 0 0</xyzOffset>
 		<rpyOffset>0 0 0</rpyOffset>
